File: Board/KiCad/USBKeyboard4S1.kicad_pcb (KiCad board)
At the start: 2 copper layers, 61 x 40.6 mm, 36 parts, among them J1 Conn_01x08, J2 USB_A, J3 Conn_01x06, J4 Conn_01x04, SW1 SW_Push_Dual, U1 PIC32MX230F064B, U2 LP2950-3.3_TO252, Y1 12MHz

Commit message: Hardware version 0.1.1
Parts:
- added C13: 22p, Capacitor_THT:C_Disc_D3.0mm_W2.0mm_P2.50mm, F.Cu at (109.3, 90.8)
- moved R6 8.89 mm to (111.8, 81.9)
- moved R7 5.45 mm to (114.3, 69.5), turned to 0 degrees
- moved R8 3.81 mm to (111.8, 74.3)
- moved R9 3.81 mm to (111.8, 78.1)
- moved D3 2.54 mm to (160.0, 74.3), turned to 180 degrees
- moved D1 2.54 mm to (148.6, 73.0), turned to -90 degrees
- moved D2 2.54 mm to (153.0, 73.0), turned to -90 degrees
- moved R4 0.13 mm to (120.1, 69.4)
Connections:
- D1 pad 1: KATA_LED -> /KATA_LED_V
- D1 pad 2: /KATA_LED_V -> KATA_LED
- D2 pad 1: HIRA_LED -> /HIRA_LED_V
- D2 pad 2: /HIRA_LED_V -> HIRA_LED
- D3 pad 1: CAPS_LED -> /CAPS_LED_V
- D3 pad 2: /CAPS_LED_V -> CAPS_LED
Routing:
- net HPP: track 36.5 -> 46.7 mm
- net +3.3V: track 248.8 -> 252.5 mm
- net GND: track 255.4 -> 258.0 mm
- net KRES2: track 34.4 -> 36.7 mm
- net KRES1: track 33.5 -> 34.9 mm, vias 0 -> 1
- net LED: track 35.2 -> 36.1 mm
- net BREAK: track 39.0 -> 39.7 mm
- net Y: track 31.8 -> 32.5 mm
Other:
- board text added: "Rev. 0.1.1"
- board text removed: "Rev. 0.1"
