File: Board/KiCad/USBKeyboard4S1.kicad_sch (KiCad schematic)
At the start: 32 parts, among them J1 Conn_01x08, J2 USB_A, J3 Conn_01x06, J4 Conn_01x04, SW1 SW_Push_Dual, U1 PIC32MX230F064B, U2 LP2950-3.3_TO252, Y1 12MHz

Commit message: Hardware version 0.1.1
Parts:
- added C13: 22p, Capacitor_THT:C_Disc_D3.0mm_W2.0mm_P2.50mm, symbol Device:C
- D1, D2, D3: symbol Device:LED -> MySymbols:LED_AK
Connections:
- net CAPS_LED: now also D3.2 (K); no longer D3.1 (K)
- net CAPS_LED_V: now also D3.1 (A); no longer D3.2 (A)
- net GND: now also C13.1
- net HIRA_LED: now also D2.2 (K); no longer D2.1 (K)
- net HIRA_LED_V: now also D2.1 (A); no longer D2.2 (A)
- net HPP: now also C13.2
- net KATA_LED: now also D1.2 (K); no longer D1.1 (K)
- net KATA_LED_V: now also D1.1 (A); no longer D1.2 (A)
Other:
- moved on the sheet: C11, C12, C9, R4, R5, SW1, Y1
